Commit message: 새로운 Yahboomcar X3 모델을 위한 SDF 파일 추가 및 URDF 파일 업데이트: 바퀴, LiDAR, 카메라 링크 및 차동 구동 시스템 포함

File: v2x_ball_bot_description/urdf/yahboomcar_X3.urdf.xacro (robot description, xacro)
@@ -1,183 +1,66 @@
-<!-- ===== XACRO ARGS (추가) ===== -->
-<xacro:arg name="ns"               default="car1"/>
-<xacro:arg name="left_joint"       default="left_wheel_joint"/>
-<xacro:arg name="right_joint"      default="right_wheel_joint"/>
-<xacro:arg name="wheel_separation" default="0.30"/>   <!-- 바퀴 간격(m), 필요 시 조정 -->
-<xacro:arg name="wheel_diameter"   default="0.10"/>   <!-- 바퀴 지름(m), 필요 시 조정 -->
-<!-- 프레임 이름: nav2/odom/tf 일관화용 -->
-<xacro:arg name="base_frame"       default="${ns}/base_link"/>
-<xacro:arg name="odom_frame"       default="${ns}/odom"/>
-<!-- LiDAR가 있다면 링크 이름(URDF상의 링크명과 정확히 일치해야 함) -->
-<xacro:arg name="laser_link_name"  default="${ns}/laser_link"/>
-<!-- 편의 프로퍼티 -->
-<xacro:property name="ns_prefix"   value="${ns}"/>
-<?xml version="1.0" encoding="utf-8"?>
-<robot name="yahboomcar" xmlns:xacro="http://wiki.ros.org/xacro">
-    <material name="Green">
-        <color rgba="0 0.7 0 1"/>
-    </material>
-    <material name="White">
-        <color rgba="0.7 0.7 0.7 1"/>
-    </material>
-    <xacro:property name="ns" value="$(arg ns)"/>
-    <link name="${ns}/base_footprint"/>
-    <link name="${ns}/imu_link"/>
-    <!-- common link-->
-    <xacro:macro name="common_link" params="name material path *origin">
-        <link name="${ns}/${name}">
-            <visual>
-                <geometry>
-                    <mesh filename="package://yahboomcar_description/meshes/${path}/${name}.STL"/>
-                </geometry>
-                <origin xyz="0 0 0" rpy="0 0 0"/>
-                <material name="${material}"/>
-            </visual>
-            <collision>
-                <geometry>
-                    <mesh filename="package://yahboomcar_description/meshes/${path}/${name}.STL"/>
-                </geometry>
-                <origin xyz="0 0 0" rpy="0 0 0"/>
-            </collision>
-            <xacro:insert_block name="origin"/>
-        </link>
-    </xacro:macro>
-    <!-- continuous joint-->
-    <xacro:macro name="continuous_joint" params="name parent child xyz rpy axis">
-        <joint name="${ns}/${name}" type="continuous">
-            <parent link="${ns}/${parent}"/>
-            <child link="${ns}/${child}"/>
-            <origin xyz="${xyz}" rpy="${rpy}"/>
-            <axis xyz="${axis}"/>
-            <limit lower="${-pi}" upper="${pi}" effort="100" velocity="1"/>
-        </joint>
-    </xacro:macro>
-    <!-- fixed joint-->
-    <xacro:macro name="fixed_joint" params="name parent child xyz rpy">
-        <joint name="${ns}/${name}" type="fixed">
-            <parent link="${ns}/${parent}"/>
-            <child link="${ns}/${child}"/>
-            <origin xyz="${xyz}" rpy="${rpy}"/>
-        </joint>
-    </xacro:macro>
-    <common_link name="base_link" material="Green" path="mecanum">
-        <inertial>
-            <origin xyz="0.00498197982182523 5.70233829969297E-05 -0.0121008098068578" rpy="0 0 0"/>
-            <mass value="0.486218814966626"/>
-            <inertia
-                    ixx="0.00196277727666921"
-                    ixy="2.50447049446755E-07"
-                    ixz="0.000140534767811098"
-                    iyy="0.00457256033711368"
-                    iyz="2.68618064993882E-07"
-                    izz="0.00493927269870476"/>
-        </inertial>
-    </common_link>
-    <fixed_joint name="base_joint" parent="base_footprint" child="base_link" xyz="0.0 0.0 0.0815" rpy="0 0 0"/>
-    <fixed_joint name="base_imu" parent="base_link" child="imu_link" xyz="-0.06 0.01 0.01" rpy="0 3.1415 1.5707"/>
-    <common_link name="front_right_wheel" material="White" path="mecanum">
-        <inertial>
-            <origin xyz="1.9051E-06 -2.3183E-07 -0.00064079" rpy="0 0 0"/>
-            <mass value="0.051532"/>
-            <inertia ixx="1.4595E-05" ixy="-4.3975E-10" ixz="4.415E-10"
-                     iyy="1.4594E-05" iyz="-1.7476E-09" izz="2.4264E-05"/>
-        </inertial>
-    </common_link>
-    <continuous_joint name="front_right_joint" parent="base_link" child="front_right_wheel"
-                      xyz="0.08 -0.0845 -0.0389" rpy="-${pi/2} 0 ${pi}" axis="0 0 1"/>
-    <common_link name="front_left_wheel" material="White" path="mecanum">
-        <inertial>
-            <origin xyz="2.3728E-06 -9.4228E-07 0.00064068" rpy="0 0 0"/>
-            <mass value="0.051543"/>
-            <inertia ixx="1.4597E-05" ixy="-4.7945E-10" ixz="-2.4786E-10"
-                     iyy="1.4598E-05" iyz="1.7972E-09" izz="2.4267E-05"/>
-        </inertial>
-    </common_link>
-    <continuous_joint name="front_left_joint" parent="base_link" child="front_left_wheel"
-                      xyz="0.08 0.084492 -0.0389" rpy="${pi/2} 0 0" axis="0 0 1"/>
-    <common_link name="back_right_wheel" material="White" path="mecanum">
-        <inertial>
-            <origin xyz="-1.75924169923403E-06 1.28388821071107E-06 -0.000590549296238266" rpy="0 0 0"/>
-            <mass value="0.051540174053366"/>
-            <inertia ixx="1.45974152250002E-05" ixy="1.94850559178397E-10" ixz="-1.61846387282284E-09"
-                     iyy="1.4596501955693E-05" iyz="-6.27904057423818E-10" izz="2.42663091380451E-05"/>
-        </inertial>
-    </common_link>
-    <continuous_joint name="back_right_joint" parent="base_link" child="back_right_wheel"
-                      xyz="-0.08 -0.0845 -0.03946" rpy="-${pi/2} 0 ${pi}" axis="0 0 1"/>
-    <common_link name="back_left_wheel" material="White" path="mecanum">
-        <inertial>
-            <origin xyz="-4.01213085227115E-07 2.04910264598596E-06 0.000590775697051377" rpy="0 0 0"/>
-            <mass value="0.0515309299357028"/>
-            <inertia ixx="1.45942986129926E-05" ixy="-3.19787215398093E-10" ixz="1.74943062058915E-09"
-                     iyy="1.45948727598913E-05" iyz="1.61769812110049E-10" izz="2.4263683888153E-05"/>
-        </inertial>
-    </common_link>
-    <continuous_joint name="back_left_joint" parent="base_link" child="back_left_wheel"
-                      xyz="-0.08 0.084492 -0.03954" rpy="${pi/2} 0 0" axis="0 0 1"/>
-    <common_link name="laser_link" material="White" path="sensor">
-        <inertial>
-            <origin xyz="-0.0176558922685589 0.000671805271544437 0.0219302095894866" rpy="0 0 0"/>
-            <mass value="0.0483909504209895"/>
-            <inertia ixx="1.58456966399128E-05" ixy="-4.23913983850005E-07" ixz="-2.09597897904374E-07"
-                     iyy="3.89262522903605E-05" iyz="3.24809725932687E-07" izz="4.86230801106223E-05"/>
-        </inertial>
-    </common_link>
-    <fixed_joint name="laser_joint" parent="base_link" child="laser_link" xyz="0.0435 5.25826986680105E-05 0.11" rpy="0 0 0"/>
-    <common_link name="camera_link" material="White" path="sensor">
-        <inertial>
-            <origin xyz="0 0 0" rpy="0 0 0"/>
-            <mass value="0"/>
-            <inertia ixx="0" ixy="0" ixz="0" iyy="0" iyz="0" izz="0"/>
-        </inertial>
-    </common_link>
-    <fixed_joint name="camera_joint" parent="base_link" child="camera_link" xyz="0.057105 1.7948E-05 0.03755" rpy="0 0 0"/>
+<?xml version="1.0"?>
+<robot name="yahboomcar_X3" xmlns:xacro="http://www.ros.org/wiki/xacro">
+  <!-- ===== XACRO ARGS ===== -->
+  <xacro:arg name="ns"               default="car1"/>
+  <xacro:property name="ns" value="$(arg ns)"/>
+  <xacro:arg name="left_joint"       default="front_left_joint"/>
+  <xacro:arg name="right_joint"      default="front_right_joint"/>
+  <xacro:arg name="wheel_separation" default="0.30"/>
+  <xacro:arg name="wheel_diameter"   default="0.10"/>
+  <xacro:arg name="base_frame"       default="${ns}/base_link"/>
+  <xacro:arg name="odom_frame"       default="${ns}/odom"/>
+  <xacro:arg name="laser_link_name"  default="${ns}/laser_link"/>
+  <!-- 재질 -->
+  <material name="Green"><color rgba="0 0.7 0 1"/></material>
+  <material name="White"><color rgba="0.7 0.7 0.7 1"/></material>
+  <!-- ===== 매크로 ===== -->
+  <xacro:macro name="common_link" params="name material path *origin">
+    <link name="${ns}/${name}">
+      <visual>
+        <geometry>
+          <mesh filename="package://v2x_ball_bot_description/meshes/${path}/${name}.STL"/>
+        </geometry>
+        <origin xyz="0 0 0" rpy="0 0 0"/>
+        <material name="${material}"/>
+      </visual>
+      <collision>
+        <geometry>
+          <mesh filename="package://v2x_ball_bot_description/meshes/${path}/${name}.STL"/>
+        </geometry>
+        <origin xyz="0 0 0" rpy="0 0 0"/>
+      </collision>
+      <xacro:insert_block name="origin"/>
+    </link>
+  </xacro:macro>
+  <xacro:macro name="continuous_joint" params="name parent child xyz rpy axis">
+    <joint name="${ns}/${name}" type="continuous">
+      <parent link="${ns}/${parent}"/>
+      <child  link="${ns}/${child}"/>
+      <origin xyz="${xyz}" rpy="${rpy}"/>
+      <axis xyz="${axis}"/>
+    </joint>
+  </xacro:macro>
+  <xacro:macro name="fixed_joint" params="name parent child xyz rpy">
+    <joint name="${ns}/${name}" type="fixed">
+      <parent link="${ns}/${parent}"/>
+      <child  link="${ns}/${child}"/>
+      <origin xyz="${xyz}" rpy="${rpy}"/>
+    </joint>
+  </xacro:macro>
+  <gazebo>
+    <plugin name="skid_steer" filename="libgazebo_ros_skid_steer_drive.so">
+      <front_left_joint> ${ns}/front_left_joint  </front_left_joint>
+      <rear_left_joint>  ${ns}/back_left_joint   </rear_left_joint>
+      <front_right_joint>${ns}/front_right_joint </front_right_joint>
+      <rear_right_joint> ${ns}/back_right_joint  </rear_right_joint>
+      <wheel_separation>$(arg wheel_separation)</wheel_separation>
+      <wheel_diameter>$(arg wheel_diameter)</wheel_diameter>
+      <odom_frame>$(arg odom_frame)</odom_frame>
+      <base_frame>$(arg base_frame)</base_frame>
+      <publish_tf>true</publish_tf>
+      <cmd_vel_topic>cmd_vel</cmd_vel_topic>
+      <odometry_topic>odom</odometry_topic>
+      <update_rate>50</update_rate>
+    </plugin>
+  </gazebo>
 </robot>
-<!-- ===== GAZEBO PLUGINS (추가) ===== -->
-<!-- 1) 조인트 상태 퍼블리셔 (RViz/TF 확인용) -->
-<gazebo>
-  <plugin name="joint_state_publisher" filename="libgazebo_ros_joint_state_publisher.so">
-    <update_rate>50</update_rate>
-  </plugin>
-</gazebo>
-<!-- 2) 차동구동 (cmd_vel -> odom/Tf) -->
-<gazebo>
-  <plugin name="diff_drive" filename="libgazebo_ros_diff_drive.so">
-    <!-- 필수: 바퀴 조인트 -->
-    <left_joint>$(arg left_joint)</left_joint>
-    <right_joint>$(arg right_joint)</right_joint>
-    <!-- 기구 파라미터 -->
-    <wheel_separation>$(arg wheel_separation)</wheel_separation>
-    <wheel_diameter>$(arg wheel_diameter)</wheel_diameter>
-    <!-- 프레임/토픽 -->
-    <odom_frame>$(arg odom_frame)</odom_frame>       <!-- 예: car1/odom -->
-    <base_frame>$(arg base_frame)</base_frame>       <!-- 예: car1/base_link -->
-    <publish_tf>true</publish_tf>
-    <cmd_vel_topic>cmd_vel</cmd_vel_topic>           <!-- 네임스페이스가 자동으로 붙습니다: /car1/cmd_vel -->
-    <odometry_topic>odom</odometry_topic>            <!-- /car1/odom -->
-    <update_rate>50</update_rate>
-  </plugin>
-</gazebo>
-<!-- 3) (선택) 2D LiDAR: laser_link_name 링크가 있을 때만 -->
-<gazebo reference="$(arg laser_link_name)">
-  <sensor type="ray" name="lidar">
-    <update_rate>10</update_rate>
-    <ray>
-      <scan>
-        <horizontal>
-          <samples>360</samples>
-          <resolution>1</resolution>
-          <min_angle>-3.14159</min_angle>
-          <max_angle> 3.14159</max_angle>
-        </horizontal>
-      </scan>
-      <range>
-        <min>0.1</min>
-        <max>8.0</max>
-      </range>
-    </ray>
-    <plugin name="gazebo_ros_ray_sensor" filename="libgazebo_ros_ray_sensor.so">
-      <frame_name>$(arg base_frame)</frame_name>
-      <topic>scan</topic> <!-- 네임스페이스 붙어서 /car1/scan 로 나갑니다 -->
-    </plugin>
-  </sensor>
-</gazebo>

Commit message: Update launch files and robot description: Modify TF nodes, add visual servoing node, and enhance URDF parameters for Yahboomcar X3 model

File: v2x_ball_bot_description/urdf/yahboomcar_X3.urdf.xacro (robot description, xacro)
@@ -1,66 +1,67 @@
 <?xml version="1.0"?>
 <robot name="yahboomcar_X3" xmlns:xacro="http://www.ros.org/wiki/xacro">
-  <!-- ===== XACRO ARGS ===== -->
-  <xacro:arg name="ns"               default="car1"/>
-  <xacro:property name="ns" value="$(arg ns)"/>
-  <xacro:arg name="left_joint"       default="front_left_joint"/>
-  <xacro:arg name="right_joint"      default="front_right_joint"/>
-  <xacro:arg name="wheel_separation" default="0.30"/>
-  <xacro:arg name="wheel_diameter"   default="0.10"/>
-  <xacro:arg name="base_frame"       default="${ns}/base_link"/>
-  <xacro:arg name="odom_frame"       default="${ns}/odom"/>
-  <xacro:arg name="laser_link_name"  default="${ns}/laser_link"/>
+  <!-- 기본 파라미터 -->
+  <xacro:property name="wheel_separation" value="0.30"/>   <!-- 좌우 바퀴 간 거리 -->
+  <xacro:property name="wheel_radius" value="0.05"/>       <!-- 바퀴 반지름 -->
+  <xacro:property name="wheel_thickness" value="0.02"/>    <!-- 바퀴 두께 -->
+  <xacro:property name="base_size_x" value="0.3"/>         <!-- 베이스 길이 -->
+  <xacro:property name="base_size_y" value="0.2"/>         <!-- 베이스 폭 -->
+  <xacro:property name="base_size_z" value="0.1"/>         <!-- 베이스 높이 -->
   <!-- 재질 -->
-  <material name="Green"><color rgba="0 0.7 0 1"/></material>
-  <material name="White"><color rgba="0.7 0.7 0.7 1"/></material>
-  <!-- ===== 매크로 ===== -->
-  <xacro:macro name="common_link" params="name material path *origin">
-    <link name="${ns}/${name}">
+  <material name="Green"><color rgba="0 1 0 1"/></material>
+  <material name="Black"><color rgba="0 0 0 1"/></material>
+  <material name="Gray"><color rgba="0.5 0.5 0.5 1"/></material>
+  <!-- ===== Base link ===== -->
+  <link name="base_link">
+    <visual>
+      <origin xyz="0 0 ${base_size_z/2}" rpy="0 0 0"/>
+      <geometry>
+        <box size="${base_size_x} ${base_size_y} ${base_size_z}"/>
+      </geometry>
+      <material name="Gray"/>
+    </visual>
+    <collision>
+      <origin xyz="0 0 ${base_size_z/2}" rpy="0 0 0"/>
+      <geometry>
+        <box size="${base_size_x} ${base_size_y} ${base_size_z}"/>
+      </geometry>
+    </collision>
+    <inertial>
+      <mass value="5.0"/>
+      <inertia ixx="0.1" iyy="0.1" izz="0.1" ixy="0.0" ixz="0.0" iyz="0.0"/>
+    </inertial>
+  </link>
+  <!-- ===== Wheels ===== -->
+  <xacro:macro name="wheel" params="name x y">
+    <link name="${name}">
       <visual>
+        <origin xyz="0 0 0" rpy="1.5708 0 0"/>
         <geometry>
-          <mesh filename="package://v2x_ball_bot_description/meshes/${path}/${name}.STL"/>
+          <cylinder radius="${wheel_radius}" length="${wheel_thickness}"/>
         </geometry>
-        <origin xyz="0 0 0" rpy="0 0 0"/>
-        <material name="${material}"/>
+        <material name="Black"/>
       </visual>
       <collision>
+        <origin xyz="0 0 0" rpy="1.5708 0 0"/>
         <geometry>
-          <mesh filename="package://v2x_ball_bot_description/meshes/${path}/${name}.STL"/>
+          <cylinder radius="${wheel_radius}" length="${wheel_thickness}"/>
         </geometry>
-        <origin xyz="0 0 0" rpy="0 0 0"/>
       </collision>
-      <xacro:insert_block name="origin"/>
+      <inertial>
+        <mass value="0.5"/>
+        <inertia ixx="0.01" iyy="0.01" izz="0.01" ixy="0.0" ixz="0.0" iyz="0.0"/>
+      </inertial>
     </link>
-  </xacro:macro>
-  <xacro:macro name="continuous_joint" params="name parent child xyz rpy axis">
-    <joint name="${ns}/${name}" type="continuous">
-      <parent link="${ns}/${parent}"/>
-      <child  link="${ns}/${child}"/>
-      <origin xyz="${xyz}" rpy="${rpy}"/>
-      <axis xyz="${axis}"/>
+    <joint name="${name}_joint" type="continuous">
+      <parent link="base_link"/>
+      <child link="${name}"/>
+      <origin xyz="${x} ${y} 0" rpy="0 0 0"/>
+      <axis xyz="0 1 0"/>
     </joint>
   </xacro:macro>
-  <xacro:macro name="fixed_joint" params="name parent child xyz rpy">
-    <joint name="${ns}/${name}" type="fixed">
-      <parent link="${ns}/${parent}"/>
-      <child  link="${ns}/${child}"/>
-      <origin xyz="${xyz}" rpy="${rpy}"/>
-    </joint>
-  </xacro:macro>
-  <gazebo>
-    <plugin name="skid_steer" filename="libgazebo_ros_skid_steer_drive.so">
-      <front_left_joint> ${ns}/front_left_joint  </front_left_joint>
-      <rear_left_joint>  ${ns}/back_left_joint   </rear_left_joint>
-      <front_right_joint>${ns}/front_right_joint </front_right_joint>
-      <rear_right_joint> ${ns}/back_right_joint  </rear_right_joint>
-      <wheel_separation>$(arg wheel_separation)</wheel_separation>
-      <wheel_diameter>$(arg wheel_diameter)</wheel_diameter>
-      <odom_frame>$(arg odom_frame)</odom_frame>
-      <base_frame>$(arg base_frame)</base_frame>
-      <publish_tf>true</publish_tf>
-      <cmd_vel_topic>cmd_vel</cmd_vel_topic>
-      <odometry_topic>odom</odometry_topic>
-      <update_rate>50</update_rate>
-    </plugin>
-  </gazebo>
+  <!-- 바퀴 4개 배치 -->
+  <xacro:wheel name="front_left_wheel"  x="${ base_size_x/2 }"  y="${ wheel_separation/2 }"/>
+  <xacro:wheel name="front_right_wheel" x="${ base_size_x/2 }"  y="-${ wheel_separation/2 }"/>
+  <xacro:wheel name="rear_left_wheel"   x="-${ base_size_x/2 }" y="${ wheel_separation/2 }"/>
+  <xacro:wheel name="rear_right_wheel"  x="-${ base_size_x/2 }" y="-${ wheel_separation/2 }"/>
 </robot>
